File: Boards/Window/Window.brd (EAGLE design)
At the start: 63.2 x 61.2 mm, 68 parts, among them IC1 LM358D, J1 ISP, Q5 FQD4N20, Q6 FQD4N20, Q7 FQD4P25, Q8 FQD4P25

Commit message: Prepared board for production, last minute error checks and rotations
Parts:
- added JP7: M01PTH_LONGPAD, 1_SparkFun-Connectors:1X01_LONGPAD
Connections:
- new net N$17: JP7.1, U$4.44
Routing:
- net N$17: track 0.00 -> 4.46 mm
- net BOTTOM_LIMIT: track 56.1 -> 59.8 mm
- net TOP_LIMIT: track 47.3 -> 51.1 mm
Changed lines of the file:
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@@
 <?xml version="1.0" encoding="utf-8"?>
 <!DOCTYPE eagle SYSTEM "eagle.dtd">
-<eagle version="7.1.0">
+<eagle version="6.6.0">
 <drawing>
 <settings>
@@
 <layers>
 <layer number="1" name="Top" color="4" fill="1" visible="yes" active="yes"/>
+<layer number="2" name="Route2" color="1" fill="3" visible="no" active="no"/>
+<layer number="3" name="Route3" color="4" fill="3" visible="no" active="no"/>
+<layer number="14" name="Route14" color="1" fill="6" visible="no" active="no"/>
+<layer number="15" name="Route15" color="4" fill="6" visible="no" active="no"/>
 <layer number="16" name="Bottom" color="1" fill="1" visible="yes" active="yes"/>
 <layer number="17" name="Pads" color="2" fill="1" visible="yes" active="yes"/>
@@
 <pass name="Default">
 <param name="RoutingGrid" value="50mil"/>
-<param name="AutoGrid" value="1"/>
-<param name="Efforts" value="0"/>
-<param name="TopRouterVariant" value="1"/>
 <param name="tpViaShape" value="round"/>
 <param name="PrefDir.1" value="|"/>
@@
 <element name="U$7" library="1_SparkFun-DigitalIC" package="SOT23-5" value="INVERTER" x="9.398" y="51.054"/>
 <element name="JP11" library="1_SparkFun-Connectors" package="1X02" value="M02PTH" x="13.97" y="49.53"/>
+<element name="JP7" library="1_SparkFun-Connectors" package="1X01_LONGPAD" value="M01PTH_LONGPAD" x="25.4" y="27.432" rot="R90"/>
 </elements>
 <signals>
@@
 <wire x1="13.716" y1="16.256" x2="11.43" y2="18.542" width="0.3048" layer="1"/>
 <wire x1="11.43" y1="18.542" x2="11.43" y2="20.574" width="0.3048" layer="1"/>
-<wire x1="11.43" y1="20.574" x2="11.176" y2="20.828" width="0.3048" layer="1"/>
-<via x="11.176" y="20.828" extent="1-16" drill="0.7" shape="square"/>
-<wire x1="11.176" y1="20.828" x2="11.176" y2="27.94" width="0.3048" layer="16"/>
+<wire x1="11.43" y1="20.574" x2="11.176" y2="21.844" width="0.3048" layer="1"/>
+<via x="11.176" y="21.844" extent="1-16" drill="0.7" shape="square"/>
+<wire x1="11.176" y1="21.844" x2="11.176" y2="27.94" width="0.3048" layer="16"/>
 <contactref element="U$4" pad="28"/>
 <wire x1="11.472" y1="34.036" x2="7.366" y2="34.036" width="0.3048" layer="1"/>
@@
 <wire x1="54.61" y1="31.242" x2="29.972" y2="31.242" width="0.3048" layer="1"/>
 <contactref element="U$4" pad="42"/>
-<wire x1="29.972" y1="31.242" x2="24.892" y2="26.162" width="0.3048" layer="1"/>
 <wire x1="19.672" y1="28.236" x2="19.672" y2="26.81" width="0.3048" layer="1"/>
-<wire x1="19.672" y1="26.81" x2="20.32" y2="26.162" width="0.3048" layer="1"/>
-<wire x1="20.32" y1="26.162" x2="24.892" y2="26.162" width="0.3048" layer="1"/>
+<wire x1="19.672" y1="26.81" x2="21.59" y2="24.892" width="0.3048" layer="1"/>
+<wire x1="21.59" y1="24.892" x2="24.638" y2="24.892" width="0.3048" layer="1"/>
+<wire x1="24.638" y1="24.892" x2="25.146" y2="25.4" width="0.3048" layer="1"/>
+<wire x1="25.146" y1="25.4" x2="28.702" y2="25.4" width="0.3048" layer="1"/>
+<wire x1="28.702" y1="25.4" x2="28.956" y2="25.654" width="0.3048" layer="1"/>
+<wire x1="28.956" y1="25.654" x2="28.956" y2="30.226" width="0.3048" layer="1"/>
+<wire x1="28.956" y1="30.226" x2="29.972" y2="31.242" width="0.3048" layer="1"/>
 </signal>
 <signal name="BOTTOM_LIMIT">
@@
 <wire x1="54.356" y1="31.75" x2="29.718" y2="31.75" width="0.3048" layer="1"/>
 <contactref element="U$4" pad="43"/>
-<wire x1="29.718" y1="31.75" x2="24.638" y2="26.67" width="0.3048" layer="1"/>
-<wire x1="24.638" y1="26.67" x2="20.828" y2="26.67" width="0.3048" layer="1"/>
 <wire x1="20.472" y1="28.236" x2="20.472" y2="27.026" width="0.3048" layer="1"/>
-<wire x1="20.472" y1="27.026" x2="20.828" y2="26.67" width="0.3048" layer="1"/>
+<wire x1="29.718" y1="31.75" x2="28.448" y2="30.48" width="0.3048" layer="1"/>
+<wire x1="28.448" y1="30.48" x2="28.448" y2="25.908" width="0.3048" layer="1"/>
+<wire x1="28.448" y1="25.908" x2="24.892" y2="25.908" width="0.3048" layer="1"/>
+<wire x1="24.892" y1="25.908" x2="24.384" y2="25.4" width="0.3048" layer="1"/>
+<wire x1="24.384" y1="25.4" x2="22.098" y2="25.4" width="0.3048" layer="1"/>
+<wire x1="22.098" y1="25.4" x2="20.472" y2="27.026" width="0.3048" layer="1"/>
 </signal>
 <signal name="TRIG">
@@
 <wire x1="1.27" y1="10.668" x2="1.27" y2="21.336" width="0.6096" layer="1"/>
 <wire x1="1.27" y1="21.336" x2="2.032" y2="22.098" width="0.6096" layer="1"/>
-<wire x1="2.032" y1="22.098" x2="2.794" y2="22.86" width="0.6096" layer="1"/>
-<wire x1="2.794" y1="22.86" x2="8.382" y2="22.86" width="0.6096" layer="1"/>
-<wire x1="8.382" y1="22.86" x2="9.144" y2="22.098" width="0.6096" layer="1"/>
-<wire x1="9.144" y1="22.098" x2="13.208" y2="22.098" width="0.6096" layer="1"/>
+<wire x1="2.032" y1="22.098" x2="3.048" y2="23.114" width="0.6096" layer="1"/>
+<wire x1="3.048" y1="23.114" x2="12.192" y2="23.114" width="0.6096" layer="1"/>
+<wire x1="12.192" y1="23.114" x2="13.208" y2="22.098" width="0.6096" layer="1"/>
 <contactref element="R15" pad="1"/>
 <contactref element="R12" pad="1"/>
@@
 <wire x1="3.68" y1="54.61" x2="4.826" y2="54.61" width="0.3048" layer="1"/>
 <wire x1="4.826" y1="54.61" x2="5.08" y2="54.356" width="0.3048" layer="1"/>
-<wire x1="5.08" y1="54.356" x2="5.08" y2="52.07" width="0.3048" layer="1"/>
-<wire x1="5.08" y1="52.07" x2="7.366" y2="49.784" width="0.3048" layer="1"/>
-<wire x1="7.366" y1="49.784" x2="7.366" y2="48.26" width="0.3048" layer="1"/>
-<wire x1="7.366" y1="48.26" x2="7.874" y2="47.752" width="0.3048" layer="1"/>
+<wire x1="5.08" y1="54.356" x2="5.08" y2="50.546" width="0.3048" layer="1"/>
+<wire x1="5.08" y1="50.546" x2="7.874" y2="47.752" width="0.3048" layer="1"/>
 <wire x1="7.874" y1="47.752" x2="9.652" y2="47.752" width="0.3048" layer="1"/>
 <wire x1="9.652" y1="47.752" x2="10.414" y2="46.99" width="0.3048" layer="1"/>
@@
 <wire x1="39.624" y1="54.102" x2="39.624" y2="54.61" width="0.3048" layer="16"/>
 </signal>
+<signal name="N$17">
+<contactref element="U$4" pad="44"/>
+<contactref element="JP7" pad="1"/>
+<wire x1="25.4" y1="27.432" x2="22.076" y2="27.432" width="0.3048" layer="1"/>
+<wire x1="22.076" y1="27.432" x2="21.272" y2="28.236" width="0.3048" layer="1"/>
+</signal>
 </signals>
