File: Boards/Window/Window.sch (EAGLE design)
At the start: 68 parts, among them IC1 LM358D, J1 ISP, Q5 FQD4N20, Q6 FQD4N20, Q7 FQD4P25, Q8 FQD4P25

Commit message: Prepared board for production, last minute error checks and rotations
Parts:
- added JP7: M01PTH_LONGPAD, 1_SparkFun-Connectors:M01PTH_LONGPAD
Connections:
- new net N$17: JP7.1, U$4.PA4(ADC4)
Changed lines of the file:
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@@
 <?xml version="1.0" encoding="utf-8"?>
 <!DOCTYPE eagle SYSTEM "eagle.dtd">
-<eagle version="7.1.0">
+<eagle version="6.6.0">
 <drawing>
 <settings>
@@
 <layers>
 <layer number="1" name="Top" color="4" fill="1" visible="no" active="no"/>
+<layer number="2" name="Route2" color="1" fill="3" visible="no" active="no"/>
+<layer number="3" name="Route3" color="4" fill="3" visible="no" active="no"/>
+<layer number="14" name="Route14" color="1" fill="6" visible="no" active="no"/>
+<layer number="15" name="Route15" color="4" fill="6" visible="no" active="no"/>
 <layer number="16" name="Bottom" color="1" fill="1" visible="no" active="no"/>
 <layer number="17" name="Pads" color="2" fill="1" visible="no" active="no"/>
@@
 <part name="GND30" library="1_SparkFun-Aesthetics" deviceset="GND" device=""/>
 <part name="JP11" library="1_SparkFun-Connectors" deviceset="M02" device="PTH"/>
+<part name="JP7" library="1_SparkFun-Connectors" deviceset="M01" device="PTH_LONGPAD"/>
 </parts>
 <sheets>
@@
 <instance part="GND30" gate="1" x="546.1" y="17.78"/>
 <instance part="JP11" gate="G$1" x="68.58" y="195.58"/>
+<instance part="JP7" gate="G$1" x="68.58" y="228.6"/>
 </instances>
 <busses>
@@
 </segment>
 </net>
+<net name="N$17" class="0">
+<segment>
+<pinref part="U$4" gate="G$1" pin="PA4(ADC4)"/>
+<wire x1="109.22" y1="228.6" x2="76.2" y2="228.6" width="0.1524" layer="91"/>
+<pinref part="JP7" gate="G$1" pin="1"/>
+</segment>
+</net>
