File: Boards/Media/vu.brd (EAGLE design)
At the start: 59.4 x 80 mm, 53 parts, among them IC1 LM3914N, IC2 LM324D, IC3 LM3914N, IC4 LM3914N, IC5 LM3914N

Commit message: Lots of prgress on media related boards.
Parts:
- R1, R10, R11, R12, R13, R14, R15, R16, R2, R3, R4, R5, R6, R7, R8, R9: device 1_SparkFun-Resistors:1206 -> 1_SparkFun-Resistors:0603-RES
- moved R12 30.0 mm to (7.11, 64.8), turned to 180 degrees
- moved R15 29.0 mm to (3.81, 70.9), turned to 0 degrees
- moved R6 19.4 mm to (23.9, 76.7), turned to 180 degrees
- moved R9 17.1 mm to (7.11, 70.9)
- moved R13 15.9 mm to (35.1, 71.9), turned to 90 degrees
- moved R5 15.0 mm to (17.3, 76.7)
- moved R3 13.3 mm to (16.3, 67.1), turned to 180 degrees
- moved R16 11.3 mm to (34.0, 66.5)
- moved R10 11.1 mm to (7.11, 66.8)
- moved R4 10.5 mm to (16.3, 72.4)
- moved R8 10.4 mm to (7.11, 72.9)
- moved R11 8.19 mm to (7.11, 68.8)
- moved R2 8.02 mm to (16.3, 69.6), turned to 180 degrees
- moved R7 6.88 mm to (23.6, 66.5)
- moved R1 5.86 mm to (19.6, 69.6), turned to 180 degrees
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Connections:
- net CH1: now also R7.2; no longer C10.1, C13.1, C2.1, R13.2
- net CH2: now also C13.1, R6.2; no longer R14.2
- net CH3: now also C2.1, R12.1; no longer R15.1
- net CH4: now also C10.1, R1.1; no longer R16.1
- net GND: now also R13.1, R14.1, R15.1, R16.1; no longer R10.1, R11.1, R12.1, R9.1
- net N$1: now also R11.2; no longer R6.2
- net N$10: now also R13.2, R3.1; no longer R12.2, R7.1
- net N$11: now also R10.1, R12.2; no longer R15.2, R5.1
- net N$12: now also R11.1, R16.2; no longer R11.2, R6.1
- net N$13: now also R7.1, R8.2; no longer R13.1, R3.2
- net N$14: now also R15.2, R9.2; no longer R10.2, R4.2
- net N$15: now also R5.1; no longer R2.1
- net N$16: now also R4.2, R6.1; no longer R1.2, R14.1
- net N$2: now also R9.1; no longer R4.1
- net N$3: now also R8.1; no longer R3.1
- net N$4: now also R10.2; no longer R5.2
- net N$5: now also R14.2, R5.2; no longer R2.2, R9.2
- net N$6: now also R4.1; no longer R1.1
- net N$7: now also R2.2; no longer R8.2
- net N$8: now also R3.2; no longer R7.2
- net N$9: now also R1.2, R2.1; no longer R16.2, R8.1
Routing:
- net CH4: track 0.00 -> 79.8 mm, vias 0 -> 4
- net CH1: track 0.00 -> 61.7 mm, vias 0 -> 1
- net CH3: track 0.00 -> 45.1 mm, vias 0 -> 2
- net CH2: track 0.00 -> 36.8 mm, vias 0 -> 2
- net N$14: track 0.00 -> 32.5 mm, vias 0 -> 2
- net N$10: track 0.00 -> 32.3 mm
- net VNEG: track 6.88 -> 25.9 mm
- net N$9: track 0.00 -> 16.4 mm
- net N$5: track 0.00 -> 14.1 mm
- net N$16: track 0.00 -> 11.9 mm
- net GND: track 37.4 -> 46.1 mm, vias 12 -> 16
- net N$12: track 0.00 -> 6.22 mm
- net N$15: track 0.00 -> 4.31 mm
- net N$3: track 0.00 -> 3.69 mm
- net N$2: track 0.00 -> 2.98 mm
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
Commit message: Final gerbers and board updates! Fixed PCB violations, now passes FreeDFM check!
Parts:
- removed C1, C11, C5, C9: (no value), 1_SparkFun-Capacitors:EIA3216
- removed C10, C8: 1uF, 1_SparkFun-Capacitors:1206
- removed D1, D3: (no value), 1_SparkFun-LED:LED_BARGAPH_10
- removed IC1, IC4: LM3914N, linear:DIL18
- removed R1, R13, R15, R2, R3, R7, R8, R9: (no value), 1_SparkFun-Resistors:0603-RES
- removed R17, R18, R21, R22: (no value), 1_SparkFun-Resistors:1206
- moved C3 31.0 mm to (40.6, 43.9)
- moved R10 31.0 mm to (7.11, 35.8)
- moved R11 31.0 mm to (7.11, 37.8)
- moved STANDOFF2 31.0 mm to (55.9, 43.9)
- moved C12 31.0 mm to (38.1, 4.57)
- moved C14 31.0 mm to (10.2, 4.57)
- moved R24 31.0 mm to (30.7, 9.40)
- moved C2 31.0 mm to (2.79, 20.3)
- moved C4 31.0 mm to (45.7, 37.6)
- moved C6 31.0 mm to (54.6, 37.6)
- moved C7 31.0 mm to (30.5, 32.5)
- moved IC2 31.0 mm to (27.4, 40.6)
- moved IC3 31.0 mm to (10.2, 18.5)
- moved IC5 31.0 mm to (38.1, 18.5)
- moved JP1 31.0 mm to (45.7, 45.2)
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Connections:
- removed net CH1: C8.1, IC2.1, R7.2
- removed net CH4: C10.1, IC2.8, R1.1
- removed net N$10: IC2.10, R13.2, R3.1
- removed net N$13: IC2.2, R7.1, R8.2
- removed net N$14: IC2.3, R15.2, R9.2
- removed net N$17: D1.19, IC1.11
- removed net N$18: D1.18, IC1.12
- removed net N$19: D1.17, IC1.13
- removed net N$20: D1.16, IC1.14
- removed net N$21: D1.15, IC1.15
- removed net N$22: D1.14, IC1.16
- removed net N$23: D1.13, IC1.17
- removed net N$24: D1.12, IC1.18
- removed net N$25: D1.11, IC1.1
- removed net N$26: D1.20, IC1.10
- removed net N$27: C8.2, IC1.5
- removed net N$28: IC1.8, R17.1, R18.2
- removed net N$29: IC1.6, IC1.7, R17.2
- removed net N$43: D3.19, IC4.11
- removed net N$44: D3.18, IC4.12
- removed net N$45: D3.17, IC4.13
- removed net N$46: D3.16, IC4.14
- removed net N$47: D3.15, IC4.15
- removed net N$48: D3.14, IC4.16
- removed net N$49: D3.13, IC4.17
- removed net N$50: D3.12, IC4.18
- removed net N$51: D3.11, IC4.1
- removed net N$52: D3.20, IC4.10
- removed net N$53: C10.2, IC4.5
- removed net N$54: IC4.6, IC4.7, R21.2
- removed net N$55: IC4.8, R21.1, R22.2
- removed net N$7: R2.2, U$1.4
- removed net N$8: R3.2, U$1.2
- removed net N$9: IC2.9, R1.2, R2.1
- net GND: no longer C1.C, C11.C, C5.C, C9.C, IC1.2, IC1.4, IC4.2, IC4.4, R13.1, R15.1, R18.1, R22.1
- net N$2: no longer R9.1
- net N$3: no longer R8.1
- net VCC: no longer C1.A, C11.A, C5.A, C9.A, D1.1, D1.10, D1.2, D1.3, D1.4, D1.5, D1.6, D1.7, D1.8, D1.9, D3.1, D3.10, D3.2, D3.3, D3.4, D3.5, D3.6, D3.7, D3.8, D3.9, IC1.3, IC1.9, IC4.3, IC4.9
Routing:
- net VCC: track 308.1 -> 183.6 mm
- net CH4: track 79.8 -> 0.00 mm, vias 4 -> 0
- net CH1: track 61.7 -> 0.00 mm, vias 1 -> 0
- net N$11: track 2.03 -> 36.2 mm, vias 0 -> 2
- net N$14: track 32.5 -> 0.00 mm, vias 2 -> 0
- net N$10: track 32.3 -> 0.00 mm
- net N$12: track 6.22 -> 38.1 mm, vias 0 -> 2
- net GND: track 46.1 -> 23.0 mm, vias 16 -> 8
- net N$9: track 16.4 -> 0.00 mm
- net N$51: track 13.8 -> 0.00 mm
- net N$25: track 13.8 -> 0.00 mm
- net N$54: track 7.04 -> 0.00 mm
- net N$28: track 6.25 -> 0.00 mm
- net N$29: track 6.15 -> 0.00 mm
- net N$55: track 6.14 -> 0.00 mm
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Other:
- board size 59.4 x 80 mm -> 59.4 x 49 mm
